File: hardware/ocxPrototype.kicad_pcb (KiCad board)
At the start: 4 copper layers, 228 x 115.4 mm, 118 parts, among them J1 J_LCD, J10 USB_C_Receptacle_USB2.0_16P, J2 ESP32_S3_DEVKIT_LEFT, J3 ESP32_S3_DEVKIT_RIGHT, J4 CTP, J5 Audio_+_-, J6 JoystickLeft, J7 JoystickRight, SW1 BTN_T_L, SW10 BTN_X, SW11 BTN_O, SW12 BTN_C, SW13 BTN_T, SW14 SW_Reset, SW15 BTN_T_R, SW16 SW_Boot, SW2 BTN_A_UP, SW3 BTN_A_R, SW4 BTN_A_L, SW5 BTN_A_DW, SW6 BTN_SLCT, SW7 BTN_VOL_-, SW8 BTN_VOL_+, SW9 BTN_HOME, U1 BT817Q, U2 USBLC6-2SC6, U4 PAM8302AAD, U5 MCP23017x-x-SO, U6 LMR51430, U7 W25Q128JVS, U8 DIO5661ST6, Y1 12MHz 18 pF

Commit message: README update + schematic PDF
Parts:
- removed the REF** at (220.0, 120.0)
- removed the REF** at (116.0, 123.0)
- removed the REF** at (40.1, 120.0)
- added C38: 100nF, Capacitor_SMD:C_0805_2012Metric_Pad1.18x1.45mm_HandSolder, F.Cu at (108.9, 61.9)
- added C39: 100nF, Capacitor_SMD:C_0805_2012Metric_Pad1.18x1.45mm_HandSolder, F.Cu at (114.9, 94.0)
- added REF**: MountingHole_3.2mm_M3, MountingHole:MountingHole_3.2mm_M3, F.Cu at (230.0, 92.0)
- added REF**: MountingHole_3.2mm_M3, MountingHole:MountingHole_3.2mm_M3, F.Cu at (26.0, 92.0)
- added REF**: MountingHole_3.2mm_M3, MountingHole:MountingHole_3.2mm_M3, F.Cu at (173.0, 122.0)
- added REF**: MountingHole_3.2mm_M3, MountingHole:MountingHole_3.2mm_M3, F.Cu at (76.0, 122.0)
- moved R4 164.6 mm to (29.7, 110.6), turned to 0 degrees
- moved C10 161.9 mm to (32.7, 109.7), turned to -90 degrees
- moved R3 157.8 mm to (35.7, 110.6), turned to 0 degrees
- moved C29 155.3 mm to (38.7, 109.7), turned to 90 degrees
- moved R13 152.8 mm to (214.9, 119.8), turned to 180 degrees
- moved J10 151.8 mm to (208.5, 126.2), turned to 0 degrees
- moved C12 150.8 mm to (41.9, 110.8), turned to 0 degrees
- moved R10 150.0 mm to (46.9, 106.1), turned to 0 degrees
- moved D2 149.8 mm to (229.9, 113.3), turned to 0 degrees
- moved C13 147.0 mm to (42.8, 113.9), turned to 90 degrees
- moved U4 144.4 mm to (48.3, 110.4), turned to 0 degrees
- moved FB2 142.9 mm to (53.2, 106.8), turned to 0 degrees
- moved R9 142.2 mm to (224.9, 113.3), turned to 180 degrees
- moved C18 140.8 mm to (56.5, 105.7), turned to 90 degrees
- moved C37 140.4 mm to (209.1, 117.2), turned to 0 degrees
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Connections:
- net Net-(J10-D+-PadA6) renamed /Power_Supply_USB/USB_C_D+
- net Net-(J10-D--PadA7) renamed /Power_Supply_USB/USB_C_D-
Routing:
- net VOL_MODE: track 59.1 -> 173.4 mm, vias 0 -> 2
- net +5V: track 317.6 -> 247.9 mm
- net /Power_Supply_USB/USB_C_D-: track 106.6 -> 68.3 mm, vias 6 -> 2
- net /Power_Supply_USB/USB_C_D+: track 103.3 -> 69.0 mm, vias 7 -> 3
- net Net-(U5-GPA5): track 33.8 -> 50.5 mm
- net Net-(U5-GPA6): track 32.9 -> 48.1 mm
- net Net-(U5-GPB0): track 41.8 -> 56.3 mm
- net Net-(U5-GPA2): track 165.8 -> 152.7 mm
- net Net-(U5-GPA1): track 182.1 -> 169.2 mm
- net Net-(U5-GPA3): track 179.9 -> 167.0 mm
- net Net-(U5-GPA0): track 188.4 -> 175.6 mm
- net Net-(U5-GPB1): track 45.0 -> 56.5 mm
- net Net-(U5-GPA4): track 161.8 -> 153.1 mm
- net JOY_L_BTN: track 121.8 -> 128.7 mm, vias 2 -> 0
- net AUDIO_L: track 113.0 -> 119.8 mm
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Other:
- board text added: "Jose Ramirez Giron"
- board text added: "OCX v1.0"
