File: hardware/ocxPrototype.kicad_sch (KiCad schematic)
At the start: 33 parts, among them J2 ESP32_S3_DEVKIT_LEFT, J3 ESP32_S3_DEVKIT_RIGHT, SW14 SW_Reset, SW16 SW_Boot, U1 BT817Q, Y1 12MHz 18 pF

Commit message: README update + schematic PDF
Parts:
- added C38: 100nF, Capacitor_SMD:C_0805_2012Metric_Pad1.18x1.45mm_HandSolder, symbol Device:C_Small
Connections:
- net +3.3V: now also C38.1
- net GND: now also C38.2
