File: hardware/power_supply_usb.kicad_sch (KiCad schematic)
At the start: 21 parts, among them J10 USB_C_Receptacle_USB2.0_16P, U2 USBLC6-2SC6, U6 LMR51430

Commit message: README update + schematic PDF
Connections:
- net USB_C_D-: now reaches J10.A7 (D-), J10.B7 (D-), R14.1, U2.3 (I/O2), U2.4 (I/O2)
- net USB_C_D+: now reaches J10.A6 (D+), J10.B6 (D+), R15.1, U2.1 (I/O1), U2.6 (I/O1)
