File: hardware/screen_ctrl.kicad_sch (KiCad schematic)
At the start: 18 parts, among them J1 J_LCD, J4 CTP, U8 DIO5661ST6

Commit message: README update + schematic PDF
Parts:
- added C39: 100nF, Capacitor_SMD:C_0805_2012Metric_Pad1.18x1.45mm_HandSolder, symbol Device:C_Small
Connections:
- net +3.3V: now also C39.1
- net GND: now also C39.2
